File: ariadne.kicad_pcb (KiCad board)
At the start: 2 copper layers, 48 parts, among them Q1 IRF5305-Reverse-Polarity, SW1 SW_DIP_x01, SW2 SW_DIP_x01, SW3 SW_DIP_x01, SW4 SW_DIP_x01, SW5 SW_DIP_x01, SW6 SW_DIP_x01, SW7 SW_DIP_x01, SW8 GB215AP, SW9 GB215AP, U1 Connector-POWER, U10 Power-Button, U11 LDH-45B-1050, U12 Bridgelux-Vero-18, U13 Bridgelux-Vero-29, U14 Meanwell-LDD-1200LW, U15 Bridgelux-Vero-18, U16 01x15_2.50mm_HEADER_PIN, U17 POTENTIOMETER, U18 Noctua-NF-A4x10-Fan, U2 Connector-LED-NILS, U20 01x15_2.50mm_HEADER_PIN, U21 01x15_2.50mm_HEADER_PIN, U22 Heatsink-NX301117, U23 Heatsink-HP20S-CALBL-001, U24 01x15_2.50mm_HEADER_PIN, U25 01x15_2.50mm_HEADER_PIN, U26 01x15_2.50mm_HEADER_PIN, U3 OKI-78SR-3.3_1.5-W36-C, U4 CT2084-ND-DIP-SWITCH, U5 ESP32-WROOM-32D, U6 Bridgelux-Vero-29, U7 OKI-78SR-5v, U8 Connector-LED, U9 Connector-LED

Commit message: finalized first pcb
Parts:
- added U19: Heatsink-HP20S-CALBL-001, ariadne:Heatsink-HP20S-CALBL-001, B.Cu at (168.0, 82.0)
- added U27: Heatsink-HP20S-CALBL-001, ariadne:Heatsink-HP20S-CALBL-001, B.Cu at (221.0, 82.0)
- added U28: Nils-Booster, Connector_JST:JST_PH_B4B-PH-K_1x04_P2.00mm_Vertical, F.Cu at (240.1, 121.8)
- moved SW2 101.8 mm to (171.8, 145.2)
- moved U8 94.8 mm to (175.0, 152.7), turned to 180 degrees
Connections:
- net GND renamed POWER-IN-
- net Net-(U16-Pad5) renamed NILS-PWM+
- U1 pad 1: +12V -> POWER-IN+
- U10 pad 2: +12V -> POWER-IN+
- U10 pad 3: +12V -> POWER-IN+
Routing:
- net POWER-IN-: track 0.00 -> 503.4 mm, vias 0 -> 2
- net +12V: track 0.00 -> 311.4 mm, vias 0 -> 3
- net +5V: track 0.00 -> 287.7 mm
- net LDD_1200_OUT-: track 0.00 -> 248.4 mm, vias 0 -> 1
- net LDD_1200_OUT+: track 0.00 -> 238.4 mm, vias 0 -> 3
- net FAN-PWM: track 0.00 -> 162.1 mm, vias 0 -> 3
- net +3V3: track 0.00 -> 133.7 mm
- net 45B_OUT+: track 0.00 -> 122.9 mm, vias 0 -> 2
- net 45B_OUT-: track 0.00 -> 122.5 mm
- net SW2: track 0.00 -> 120.8 mm
- net SW1: track 0.00 -> 113.9 mm, vias 0 -> 1
- net NILS-PWM+: track 0.00 -> 113.6 mm
- net SW3: track 0.00 -> 99.8 mm, vias 0 -> 2
- net LDD_1200-DIM: track 0.00 -> 84.5 mm, vias 0 -> 1
- net SW4: track 0.00 -> 79.2 mm
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- added copper zone on B.Cu, net (none)
- added copper zone on F.Cu, net (none)
- added copper zone on B.Cu, net GND
- added copper zone on F.Cu, net GND
- added copper zone on B.Cu, net Net-(U6-Pad0)
- added copper zone on F.Cu, net Net-(U6-Pad0)
Other:
- board outline added: 250 x 232 mm
- net class Power added: clearance 0.2, trace_width 1.75, via_dia 1.5, via_drill 1.2
- board text added: "Area drawn both in Cu and Mask layers"
- board text added: "Area drawn both in Mask layers but not in Cu"
- board text added: "Area drawn in both Cu but not in Mask layers"
- board text added: "Area drawn only in Cu layers"
- board text added: "Area drawn only in Mask layers"
- board text added: "GND Area"
- board text added: "Keepout area drawn both in Cu layers"
- board text added: "No area"
- board text added: "Notes:"
- board text added: "Power Check Via"
- board text added: "Power Check Via 12V"
- board text added: "Power Check Via 45B OUT+"
- board text added: "Power Check Via LDD OUT+"

Commit message: second version, in progress
Parts:
- removed the SW1 at (217.0, 140.0)
- removed the SW2 at (171.8, 145.2)
- removed SW3, SW4, SW5, SW6, SW7: SW_DIP_x01, Button_Switch_THT:SW_DIP_SPSTx01_Slide_9.78x4.72mm_W7.62mm_P2.54mm
- removed the U12 at (168.0, 82.0)
- removed the U17 at (109.0, 194.0)
- removed the U19 at (168.0, 82.0)
- removed the U22 at (109.0, 67.0)
- removed U27: Heatsink-HP20S-CALBL-001, ariadne:Heatsink-HP20S-CALBL-001
- removed U28: Nils-Booster, Connector_JST:JST_PH_B4B-PH-K_1x04_P2.00mm_Vertical
- removed the U7 at (226.0, 162.0)
- removed the U9 at (156.0, 177.0)
- added C1: CP1_Small, Capacitor_THT:CP_Radial_D5.0mm_P2.00mm, F.Cu at (-85.0, 21.0)
- added Murata-Ceramic-Capacitor-50v1-22uF1: C, Capacitor_THT:C_Disc_D3.0mm_W1.6mm_P2.50mm, F.Cu at (-67.3, 19.3)
- added Murata-Ceramic-Capacitor-50v1-22uF2: C, Capacitor_THT:C_Disc_D3.0mm_W1.6mm_P2.50mm, F.Cu at (-73.5, 22.7)
- added Murata-Ceramic-Capacitor-50v1-22uF3: C, Capacitor_THT:C_Disc_D3.0mm_W1.6mm_P2.50mm, F.Cu at (-61.6, 16.9)
- added Murata-Ceramic-Capacitor-50v1-22uF4: C, Capacitor_THT:C_Disc_D3.0mm_W1.6mm_P2.50mm, F.Cu at (-79.2, 22.7)
- added Murata-Ceramic-Capacitor-50v1-22uF5: C, Capacitor_THT:C_Disc_D3.0mm_W1.6mm_P2.50mm, F.Cu at (-67.3, 16.1)
- added Murata-Ceramic-Capacitor-50v1-22uF6: C, Capacitor_THT:C_Disc_D3.0mm_W1.6mm_P2.50mm, F.Cu at (14.1, -36.6)
- added Q2: MMBT3904, Package_TO_SOT_SMD:SOT-23, F.Cu at (-24.7, 2.23)
- added R12: R, Resistor_THT:R_Axial_DIN0204_L3.6mm_D1.6mm_P7.62mm_Horizontal, F.Cu at (-96.5, 16.1)
- added R7: R, Resistor_THT:R_Axial_DIN0204_L3.6mm_D1.6mm_P7.62mm_Horizontal, F.Cu at (-25.5, -1.62)
- added R8: R, Resistor_THT:R_Axial_DIN0204_L3.6mm_D1.6mm_P7.62mm_Horizontal, F.Cu at (-96.5, 22.4)
- added R9: R, Resistor_THT:R_Axial_DIN0204_L3.6mm_D1.6mm_P7.62mm_Horizontal, F.Cu at (-85.9, 16.1)
- added U18: Meanwell-LDD-1200LW-connector, Connector_Molex:Molex_Micro-Fit_3.0_43650-0300_1x03_P3.00mm_Horizontal, F.Cu at (70.5, -81.3)
- added U20: Meanwell-LDD-1200LW-connector, Connector_Molex:Molex_Micro-Fit_3.0_43650-0300_1x03_P3.00mm_Horizontal, F.Cu at (-37.3, 6.75)
- added U3: LDH-45B-1050-connector-master, Connector_Molex:Molex_Micro-Fit_3.0_43650-0500_1x05_P3.00mm_Horizontal, F.Cu at (-37.3, -5.20)
- added U4: Connector-LED, Connector_JST:JST_PH_B2B-PH-K_1x02_P2.00mm_Vertical, F.Cu at (-73.8, 17.3)
- added U5: OKI-78SR-12v, Converter_DCDC:Converter_DCDC_muRata_OKI-78SR_Vertical, F.Cu at (-106.5, 20.5)
- R6: value 33k -> R
- U11: value LDH-45B-1050 -> Noctua-NF-A4x10-Fan-mech; footprint OpenCelluloid:MeanWell-LDH-45B-1050 -> ariadne:Noctua-NF-A4x10
- U13: value Bridgelux-Vero-29 -> Bridgelux-Vero-29-mech; footprint ariadne:Vero-29 -> ariadne:Vero-29-mech
- U14: renamed from U18; footprint ariadne:Noctua-NF-A4x10 -> Connector_Molex:Molex_Micro-Fit_3.0_43650-0400_1x04_P3.00mm_Horizontal
- U15: value Bridgelux-Vero-18 -> Bridgelux-Vero-18-mech; footprint ariadne:Vero-18 -> ariadne:Vero-18-mech
- U2: value Connector-LED-NILS -> LDH-45B-1050-connector-slave; footprint Connector_JST:JST_PH_B2B-PH-K_1x02_P2.00mm_Vertical -> Connector_Molex:Molex_Micro-Fit_3.0_43650-0500_1x05_P3.00mm_Horizontal
- U23: value Heatsink-HP20S-CALBL-001 -> Connector-LED; footprint ariadne:Heatsink-HP20S-CALBL-001 -> Connector_JST:JST_PH_B2B-PH-K_1x02_P2.00mm_Vertical; moved to F.Cu
- U6: value Bridgelux-Vero-29 -> OKI-78SR-5v; footprint ariadne:Vero-29 -> Converter_DCDC:Converter_DCDC_muRata_OKI-78SR_Vertical
- U8: value Connector-LED -> LDH-45B-1050-mech; footprint Connector_JST:JST_PH_B2B-PH-K_1x02_P2.00mm_Vertical -> OpenCelluloid:MeanWell-LDH-45B-1050
- moved U6 344.9 mm to (-118.4, 20.5), turned to 0 degrees
- moved U23 297.1 mm to (-38.7, 11.5), turned to 0 degrees
- moved R6 281.6 mm to (-96.5, 19.3)
- moved U8 279.7 mm to (-14.5, -53.0), turned to 0 degrees
- moved U2 252.7 mm to (16.8, -40.2), turned to 0 degrees
- moved U15 241.4 mm to (-70.3, -64.8), turned to 0 degrees
- moved U11 230.8 mm to (45.6, -70.7), turned to 0 degrees
- moved U13 195.9 mm to (-70.3, -11.9)
- renumbered D2 to D1, D1 to D2, R7 to R10, R8 to R11, R9 to R13, R10 to R14, SW8 to SW1, SW9 to SW2, U3 to U10, U16 to U12, U5 to U16, U20 to U17, U21 to U19, U24 to U21, U25 to U22, U14 to U24, U26 to U25, U10 to U7, U4 to U9
Connections:
- D1 pad 1: +12V -> VIN+Master
- Q1 pad 3: +12V -> VIN+Master
- R10 pad 1: +5V -> +3V3
- R11 pad 1: +5V -> +3V3
- R6 pad 2: +5V -> FAN-PWM
- U10 pad 1: +12V -> VIN+Master
- U11 pad 1: LDH_45B-DIM -> (no net)
- U11 pad 2: POTI-45-B -> (no net)
- U11 pad 3: POWER-IN- -> (no net)
- U14 pad 1: FAN-PWM -> POWER-IN-
- U14 pad 2: POWER-IN- -> +12V
- U14 pad 3: +12V -> Net-(R12-Pad1)
- U2 pad 1: Net-(SW6-Pad1) -> Net-(U2-Pad1)
- U2 pad 2: LDD_1200_OUT- -> Net-(U2-Pad2)
- U24 pad 1: +12V -> Net-(U18-Pad1)
- U24 pad 2: POWER-IN- -> Net-(U18-Pad2)
- U24 pad 3: LDD_1200-DIM -> Net-(U18-Pad3)
- U6 pad 1: Net-(SW1-Pad2) -> VIN+Master
- U6 pad 2: 45B_OUT- -> POWER-IN-
- U8 pad 1: Net-(SW2-Pad2) -> Net-(U2-Pad1)
- U8 pad 2: 45B_OUT- -> Net-(U2-Pad2)
Routing:
- net +12V: track 311.4 -> 217.1 mm, vias 3 -> 0
- net VIN+Master: track 0.00 -> 94.4 mm, vias 0 -> 3
- net Net-(R6-Pad1): track 0.00 -> 11.3 mm
- net Net-(Q2-Pad1): track 11.3 -> 0.00 mm

Commit message: second version ready for layout
Parts:
- added REF**: MountingHole_4.3mm_M4_Pad_Via, MountingHole:MountingHole_4.3mm_M4_Pad_Via, F.Cu at (374.0, -2.50)
- added U26: SWITCH_ROCKER-300DP3J1BLKM6QE, ariadne:SWITCH_ROCKER-300DP3J1BLKM6QE, F.Cu at (-35.8, -13.4)
- added U27: LDH-65B-connector-master, Connector_Molex:Molex_Micro-Fit_3.0_43650-0400_1x04_P3.00mm_Horizontal, F.Cu at (-74.9, 36.3)
- added U28: Connector-LED, Connector_JST:JST_PH_B2B-PH-K_1x02_P2.00mm_Vertical, F.Cu at (373.0, 104.5)
- added U29: LDH-65B-mech, ariadne:MeanWell-LDH-65, F.Cu at (357.5, 60.0)
- Q1: footprint ariadne:IRF5305 -> Package_TO_SOT_THT:TO-220-3_Horizontal_TabDown
- Q2: footprint Package_TO_SOT_SMD:SOT-23 -> Package_TO_SOT_THT:TO-92
- U1: value Connector-POWER -> POWER_CONNECTOR-DCJ250-20-B-K1-A; footprint OpenCelluloid:WAGO_PCB_Klemme_2Pol -> ariadne:POWER_JACK_DCJ250-20-B-K1-A
- U24: moved to F.Cu
- U7: value Power-Button -> LDH-65B-connector-master; footprint OpenCelluloid:WAGO_PCB_Klemme_3Pol -> Connector_Molex:Molex_Micro-Fit_3.0_43650-0400_1x04_P3.00mm_Horizontal
- U8: footprint OpenCelluloid:MeanWell-LDH-45B-1050 -> ariadne:MeanWell-LDH-45B-1050-ariadne
- moved D1 407.7 mm to (-182.7, 67.6)
- moved U16 380.3 mm to (-157.2, 41.0)
- moved U19 362.2 mm to (-42.7, -59.4)
- moved SW1 350.0 mm to (-86.7, 60.5)
- moved R4 347.0 mm to (-140.6, 67.3)
- moved U17 346.1 mm to (-38.0, -59.4)
- moved R11 345.1 mm to (-14.8, -19.6)
- moved Q1 344.4 mm to (-87.6, 34.7), turned to 0 degrees
- moved R10 341.3 mm to (-27.9, -5.32), turned to 0 degrees
- moved U10 336.1 mm to (-74.9, 44.3), turned to 0 degrees
- moved SW2 333.3 mm to (-23.4, -1.94), turned to 0 degrees
- moved U12 327.4 mm to (-47.3, -59.4)
- moved U1 324.8 mm to (-22.8, -16.6), turned to 0 degrees
- moved R1 319.7 mm to (-89.3, 54.0), turned to 0 degrees
- moved R3 313.5 mm to (-98.4, 67.3)
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Connections:
- net Net-(U16-Pad24) renamed LDH-65B-DIM
- U16 pad 17: Net-(U16-Pad17) -> BOARD_GND
- U17 pad 14: Net-(U16-Pad17) -> BOARD_GND
- U3 pad 1: LDH_45B-DIM -> VIN+Master
- U3 pad 2: Net-(U3-Pad2) -> POWER-IN-
- U3 pad 3: POWER-IN- -> BOARD_GND
- U3 pad 4: POWER-IN- -> Net-(U3-Pad4)
- U3 pad 5: VIN+Master -> LDH_45B-DIM
- U7 pad 1: Net-(Q1-Pad2) -> Net-(U29-Pad1)
- U7 pad 2: POWER-IN+ -> Net-(U29-Pad2)
- U7 pad 3: POWER-IN+ -> Net-(U29-Pad3)
- U7 pad 4: (no net) -> Net-(U29-Pad4)
Routing:
- net POWER-IN-: track 503.4 -> 0.00 mm, vias 2 -> 0
- net (no net): track 0.00 -> 320.0 mm
- net +5V: track 287.7 -> 0.00 mm
- net LDD_1200_OUT-: track 248.4 -> 0.00 mm, vias 1 -> 0
- net LDD_1200_OUT+: track 238.4 -> 0.00 mm, vias 3 -> 0
- net +12V: track 217.1 -> 0.00 mm
- net FAN-PWM: track 162.1 -> 0.00 mm, vias 3 -> 0
- net +3V3: track 133.7 -> 0.00 mm
- net 45B_OUT+: track 122.9 -> 0.00 mm, vias 2 -> 0
- net 45B_OUT-: track 122.5 -> 0.00 mm
- net SW2: track 120.8 -> 0.00 mm
- net SW1: track 113.9 -> 0.00 mm, vias 1 -> 0
- net NILS-PWM+: track 113.6 -> 0.00 mm
- net SW3: track 99.8 -> 0.00 mm, vias 2 -> 0
- net VIN+Master: track 94.4 -> 0.00 mm, vias 3 -> 0
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- removed copper zone on B.Cu, net GND
Other:
- board outline removed
- board text removed: "Power Check Via LDD OUT+"

Commit message: Second version ordered
Parts:
- removed the REF** at (374.0, -2.50)
- removed U21, U22, U25: 01x15_2.50mm_HEADER_PIN, Connector_PinHeader_2.54mm:PinHeader_1x15_P2.54mm_Vertical
- added J1: Conn_01x05_Male, Connector_PinHeader_2.54mm:PinHeader_1x05_P2.54mm_Vertical, F.Cu at (138.5, 52.5)
- added J2: Conn_01x05_Male, Connector_PinHeader_2.54mm:PinHeader_1x05_P2.54mm_Vertical, F.Cu at (142.1, 52.5)
- added J3: Conn_01x05_Male, Connector_PinHeader_2.54mm:PinHeader_1x05_P2.54mm_Vertical, F.Cu at (145.4, 52.5)
- added J4: Conn_01x05_Male, Connector_PinHeader_2.54mm:PinHeader_1x05_P2.54mm_Vertical, F.Cu at (134.6, 52.6)
- added REF**: MountingHole_4.3mm_M4_Pad_Via, MountingHole:MountingHole_4.3mm_M4_Pad_Via, F.Cu at (320.2, 136.2)
- added REF**: MountingHole_4.3mm_M4_Pad_Via, MountingHole:MountingHole_4.3mm_M4_Pad_Via, F.Cu at (220.2, 223.8)
- added REF**: MountingHole_4.3mm_M4_Pad_Via, MountingHole:MountingHole_4.3mm_M4_Pad_Via, F.Cu at (132.8, 223.8)
- added REF**: MountingHole_4.3mm_M4_Pad_Via, MountingHole:MountingHole_4.3mm_M4_Pad_Via, F.Cu at (220.2, 136.2)
- added REF**: MountingHole_4.3mm_M4_Pad_Via, MountingHole:MountingHole_4.3mm_M4_Pad_Via, F.Cu at (320.2, 123.8)
- added REF**: MountingHole_4.3mm_M4_Pad_Via, MountingHole:MountingHole_4.3mm_M4_Pad_Via, F.Cu at (232.8, 36.2)
- added REF**: MountingHole_4.3mm_M4_Pad_Via, MountingHole:MountingHole_4.3mm_M4_Pad_Via, F.Cu at (232.8, 123.8)
- added REF**: MountingHole_4.3mm_M4_Pad_Via, MountingHole:MountingHole_4.3mm_M4_Pad_Via, F.Cu at (320.2, 36.2)
- added REF**: MountingHole_4.3mm_M4_Pad_Via, MountingHole:MountingHole_4.3mm_M4_Pad_Via, F.Cu at (112.0, 115.5)
- added REF**: MountingHole_4.3mm_M4_Pad_Via, MountingHole:MountingHole_4.3mm_M4_Pad_Via, F.Cu at (112.0, 44.5)
- added REF**: MountingHole_4.3mm_M4_Pad_Via, MountingHole:MountingHole_4.3mm_M4_Pad_Via, F.Cu at (41.0, 115.5)
- added REF**: MountingHole_4.3mm_M4_Pad_Via, MountingHole:MountingHole_4.3mm_M4_Pad_Via, F.Cu at (232.8, 223.8)
- added REF**: MountingHole_4.3mm_M4_Pad_Via, MountingHole:MountingHole_4.3mm_M4_Pad_Via, F.Cu at (41.0, 44.5)
- added REF**: MountingHole_4.3mm_M4_Pad_Via, MountingHole:MountingHole_4.3mm_M4_Pad_Via, F.Cu at (212.0, 115.5)
- added REF**: MountingHole_4.3mm_M4_Pad_Via, MountingHole:MountingHole_4.3mm_M4_Pad_Via, F.Cu at (141.0, 115.5)
- added REF**: MountingHole_4.3mm_M4_Pad_Via, MountingHole:MountingHole_4.3mm_M4_Pad_Via, F.Cu at (212.0, 44.5)
- added REF**: MountingHole_4.3mm_M4_Pad_Via, MountingHole:MountingHole_4.3mm_M4_Pad_Via, F.Cu at (141.0, 44.5)
- added REF**: MountingHole_4.3mm_M4_Pad_Via, MountingHole:MountingHole_4.3mm_M4_Pad_Via, F.Cu at (220.2, 123.8)
- added REF**: MountingHole_4.3mm_M4_Pad_Via, MountingHole:MountingHole_4.3mm_M4_Pad_Via, F.Cu at (132.8, 123.8)
- added REF**: MountingHole_4.3mm_M4_Pad_Via, MountingHole:MountingHole_4.3mm_M4_Pad_Via, F.Cu at (220.2, 36.2)
- added REF**: MountingHole_4.3mm_M4_Pad_Via, MountingHole:MountingHole_4.3mm_M4_Pad_Via, F.Cu at (132.8, 36.2)
- added REF**: MountingHole_4.3mm_M4_Pad_Via, MountingHole:MountingHole_4.3mm_M4_Pad_Via, F.Cu at (320.2, 223.8)
- added REF**: MountingHole_4.3mm_M4_Pad_Via, MountingHole:MountingHole_4.3mm_M4_Pad_Via, F.Cu at (232.8, 136.2)
- added REF**: MountingHole_4.3mm_M4_Pad_Via, MountingHole:MountingHole_4.3mm_M4_Pad_Via, F.Cu at (41.0, 144.5)
- added REF**: MountingHole_4.3mm_M4_Pad_Via, MountingHole:MountingHole_4.3mm_M4_Pad_Via, F.Cu at (41.0, 215.5)
- added REF**: MountingHole_4.3mm_M4_Pad_Via, MountingHole:MountingHole_4.3mm_M4_Pad_Via, F.Cu at (112.0, 144.5)
- added REF**: MountingHole_4.3mm_M4_Pad_Via, MountingHole:MountingHole_4.3mm_M4_Pad_Via, F.Cu at (112.0, 215.5)
- added REF**: MountingHole_4.3mm_M4_Pad_Via, MountingHole:MountingHole_4.3mm_M4_Pad_Via, F.Cu at (132.8, 136.2)
- D1: value D_Schottky -> D_Zener
- U11: footprint ariadne:Noctua-NF-A4x10 -> ariadne:Noctua-NF-A4x10-mech
- U14: footprint Connector_Molex:Molex_Micro-Fit_3.0_43650-0400_1x04_P3.00mm_Horizontal -> Connector_PinHeader_2.54mm:PinHeader_1x04_P2.54mm_Vertical
- U19: value 01x15_2.50mm_HEADER_PIN -> Noctua-NF-A4x10-Fan-mech-ariadne; footprint Connector_PinHeader_2.54mm:PinHeader_1x15_P2.54mm_Vertical -> ariadne:Noctua-NF-A4x10-mech
- moved U2 553.1 mm to (322.4, 164.9), turned to 90 degrees
- moved U3 424.4 mm to (223.5, 66.0), turned to 90 degrees
- moved D1 395.2 mm to (212.5, 63.5), turned to 90 degrees
- moved U4 388.8 mm to (287.4, 223.9)
- moved U6 370.6 mm to (189.5, 58.5), turned to 180 degrees
- moved U16 335.7 mm to (173.5, 99.0)
- moved R6 335.1 mm to (201.5, 116.0), turned to 180 degrees
- moved R7 305.9 mm to (194.5, 106.0)
- moved U11 305.9 mm to (76.5, 180.0)
- moved U23 304.5 mm to (182.5, 220.0), turned to 180 degrees
- moved U27 302.7 mm to (223.5, 87.0), turned to 90 degrees
- moved U24 298.8 mm to (182.5, 178.0)
- moved R1 296.6 mm to (207.2, 56.9), turned to 90 degrees
- moved U20 292.6 mm to (223.5, 104.0), turned to 90 degrees
- moved R4 291.7 mm to (150.0, 92.0), turned to 270 degrees
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Routing:
- net POWER-IN-: track 0.00 -> 270.5 mm, vias 0 -> 1
- net (no net): track 320.0 -> 91.5 mm
- net +12V: track 0.00 -> 150.3 mm, vias 0 -> 1
- net VIN+Master: track 0.00 -> 143.0 mm
- net +5V: track 0.00 -> 141.2 mm, vias 0 -> 1
- net BOARD_GND: track 0.00 -> 133.8 mm
- net +3V3: track 0.00 -> 132.9 mm, vias 0 -> 2
- net LDH_45B-DIM: track 0.00 -> 84.3 mm
- net LDD_1200-DIM: track 0.00 -> 80.3 mm, vias 0 -> 1
- net BUTTON1: track 0.00 -> 76.0 mm
- net Net-(U2-Pad1): track 0.00 -> 73.0 mm
- net BUTTON2: track 0.00 -> 72.5 mm, vias 0 -> 3
- net Net-(U29-Pad1): track 0.00 -> 71.7 mm
- net FAN-PWM: track 0.00 -> 53.1 mm
- net Net-(U29-Pad2): track 0.00 -> 52.7 mm
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- added copper zone on B.Cu, net Net-(U15-Pad0)
- added copper zone on F.Cu, net Net-(U15-Pad0)
- added copper zone on B.Cu, net POWER-IN-
- removed copper zone on F.Cu, net (none)
- removed copper zone on F.Cu, net GND
- removed copper zone on B.Cu, net Net-(U13-Pad0)
- removed copper zone on B.Cu, net Net-(U6-Pad0)
- removed copper zone on F.Cu, net Net-(U6-Pad0)
Other:
- board outline added: 300 x 200 mm
- board text added: "12V"
- board text added: "3.3V"
- board text added: "5V"
- board text removed: "Area drawn both in Cu and Mask layers"
- board text removed: "Area drawn both in Mask layers but not in Cu"
- board text removed: "Area drawn in both Cu but not in Mask layers"
- board text removed: "Area drawn only in Cu layers"
- board text removed: "Area drawn only in Mask layers"
- board text removed: "GND Area"
- board text removed: "Keepout area drawn both in Cu layers"
- board text removed: "No area"
- board text removed: "Notes:"
- board text removed: "Power Check Via"
- board text removed: "Power Check Via 12V"
- board text removed: "Power Check Via 45B OUT+"
