File: ariadne.sch (KiCad schematic (older format))
At the start: 48 parts, among them Q1 IRF5305-Reverse-Polarity, SW1 SW_DIP_x01, SW2 SW_DIP_x01, SW3 SW_DIP_x01, SW4 SW_DIP_x01, SW5 SW_DIP_x01, SW6 SW_DIP_x01, SW7 SW_DIP_x01, SW8 GB215AP, SW9 GB215AP, U1 Connector-POWER, U10 Power-Button, U11 LDH-45B-1050, U12 Bridgelux-Vero-18, U13 Bridgelux-Vero-29, U14 Meanwell-LDD-1200LW, U15 Bridgelux-Vero-18, U16 01x15_2.50mm_HEADER_PIN, U17 POTENTIOMETER, U18 Noctua-NF-A4x10-Fan, U2 Connector-LED-NILS, U20 01x15_2.50mm_HEADER_PIN, U21 01x15_2.50mm_HEADER_PIN, U22 Heatsink-NX301117, U23 Heatsink-HP20S-CALBL-001, U24 01x15_2.50mm_HEADER_PIN, U25 01x15_2.50mm_HEADER_PIN, U26 01x15_2.50mm_HEADER_PIN, U3 OKI-78SR-3.3_1.5-W36-C, U4 CT2084-ND-DIP-SWITCH, U5 ESP32-WROOM-32D, U6 Bridgelux-Vero-29, U7 OKI-78SR-5v, U8 Connector-LED, U9 Connector-LED

Commit message: finalized first pcb
Parts:
- added U19, U27: Heatsink-HP20S-CALBL-001, ariadne:Heatsink-HP20S-CALBL-001, symbol ariadne:Heatsink-HP20S-CALBL-001
- added U28: Nils-Booster, Connector_JST:JST_PH_B4B-PH-K_1x04_P2.00mm_Vertical, symbol ariadne:Nils-Booster
Connections:
- net labels added: NILS-PWM+, POWER-IN+, POWER-IN-
- wire segments 164 -> 170
Changed lines of the file:
@@
 $EndComp
-$Comp
-L power:+12V #PWR05
-U 1 1 5F871F05
-P 1550 1050
-F 0 "#PWR05" H 1550 900 50  0001 C CNN
-F 1 "+12V" H 1565 1223 50  0000 C CNN
-F 2 "" H 1550 1050 50  0001 C CNN
-F 3 "" H 1550 1050 50  0001 C CNN
-	1    1550 1050
-	0    1    1    0
-$EndComp
-Wire Wire Line
-	1550 1050 1550 1400
-$Comp
-L power:GND #PWR02
-U 1 1 5F8727DD
-P 1150 1050
-F 0 "#PWR02" H 1150 800 50  0001 C CNN
-F 1 "GND" H 1155 877 50  0000 C CNN
-F 2 "" H 1150 1050 50  0001 C CNN
-F 3 "" H 1150 1050 50  0001 C CNN
-	1    1150 1050
-	0    1    1    0
-$EndComp
-Wire Wire Line
-	1150 1050 1150 1350
 $Comp
 L power:PWR_FLAG #FLG01
 U 1 1 5F872FD4
-P 1150 1350
-F 0 "#FLG01" H 1150 1425 50  0001 C CNN
-F 1 "PWR_FLAG" H 1150 1523 50  0000 C CNN
-F 2 "" H 1150 1350 50  0001 C CNN
-F 3 "~" H 1150 1350 50  0001 C CNN
-	1    1150 1350
+P 1150 3550
+F 0 "#FLG01" H 1150 3625 50  0001 C CNN
+F 1 "PWR_FLAG" H 1150 3723 50  0000 C CNN
+F 2 "" H 1150 3550 50  0001 C CNN
+F 3 "~" H 1150 3550 50  0001 C CNN
+	1    1150 3550
 	0    -1   -1   0
 $EndComp
-Connection ~ 1150 1350
-Wire Wire Line
-	1150 1350 1150 1500
 $Comp
 L power:PWR_FLAG #FLG02
 U 1 1 5F8731D6
-P 1550 1400
-F 0 "#FLG02" H 1550 1475 50  0001 C CNN
-F 1 "PWR_FLAG" H 1550 1573 50  0000 C CNN
-F 2 "" H 1550 1400 50  0001 C CNN
-F 3 "~" H 1550 1400 50  0001 C CNN
-	1    1550 1400
+P 1850 3650
+F 0 "#FLG02" H 1850 3725 50  0001 C CNN
+F 1 "PWR_FLAG" H 1850 3823 50  0000 C CNN
+F 2 "" H 1850 3650 50  0001 C CNN
+F 3 "~" H 1850 3650 50  0001 C CNN
+	1    1850 3650
 	0    1    1    0
 $EndComp
-Connection ~ 1550 1400
-Wire Wire Line
-	1550 1400 1550 1500
 $Comp
 L OpenSourceCelluloid:Power-Button U10
@@
 $EndComp
 Wire Wire Line
-	1150 3900 1150 2950
+	1150 3900 1150 3550
 Connection ~ 1150 1500
 $Comp
@@
 Connection ~ 1850 3300
 Wire Wire Line
-	1850 3300 1850 3900
+	1850 3300 1850 3650
 Wire Wire Line
 	1550 3300 1550 2950
@@
 Wire Wire Line
 	2000 5000 1800 5000
+$Comp
+L ariadne:Heatsink-HP20S-CALBL-001 U19
+U 1 1 5F89CD06
+P 13650 3400
+F 0 "U19" H 13928 3388 50  0000 L CNN
+F 1 "Heatsink-HP20S-CALBL-001" H 13928 3297 50  0000 L CNN
+F 2 "ariadne:Heatsink-HP20S-CALBL-001" H 13650 3400 50  0001 C CNN
+F 3 "" H 13650 3400 50  0001 C CNN
+	1    13650 3400
+	1    0    0    -1
+$EndComp
+$Comp
+L ariadne:Heatsink-HP20S-CALBL-001 U27
+U 1 1 5F8A28CA
+P 14050 2200
+F 0 "U27" H 14328 2188 50  0000 L CNN
+F 1 "Heatsink-HP20S-CALBL-001" H 14328 2097 50  0000 L CNN
+F 2 "ariadne:Heatsink-HP20S-CALBL-001" H 14050 2200 50  0001 C CNN
+F 3 "" H 14050 2200 50  0001 C CNN
+	1    14050 2200
+	1    0    0    -1
+$EndComp
+$Comp
+L ariadne:Nils-Booster U28
+U 1 1 5F8A9E07
+P 13350 5800
+F 0 "U28" H 13678 5904 50  0000 L CNN
+F 1 "Nils-Booster" H 13678 5813 50  0000 L CNN
+F 2 "Connector_JST:JST_PH_B4B-PH-K_1x04_P2.00mm_Vertical" H 13350 5800 50  0001 C CNN
+F 3 "" H 13350 5800 50  0001 C CNN
+	1    13350 5800
+	1    0    0    -1
+$EndComp
+$Comp
+L power:+12V #PWR0101
+U 1 1 5F8AA130
+P 13150 5400
+F 0 "#PWR0101" H 13150 5250 50  0001 C CNN
+F 1 "+12V" H 13165 5573 50  0000 C CNN
+F 2 "" H 13150 5400 50  0001 C CNN
+F 3 "" H 13150 5400 50  0001 C CNN
+	1    13150 5400
+	1    0    0    -1
+$EndComp
+Wire Wire Line
+	13150 5400 13150 5550
+Text GLabel 8700 1350 0    50   Input ~ 0
+NILS-PWM+
+Text GLabel 13300 5300 1    50   Input ~ 0
+NILS-PWM+
+Wire Wire Line
+	13300 5300 13300 5550
+$Comp
+L power:GND #PWR0102
+U 1 1 5F8BA604
+P 13450 5300
+F 0 "#PWR0102" H 13450 5050 50  0001 C CNN
+F 1 "GND" H 13455 5127 50  0000 C CNN
+F 2 "" H 13450 5300 50  0001 C CNN
+F 3 "" H 13450 5300 50  0001 C CNN
+	1    13450 5300
+	-1   0    0    1
+$EndComp
+Wire Wire Line
+	13450 5300 13450 5400
+Wire Wire Line
+	13450 5400 13600 5400
+Wire Wire Line
+	13600 5400 13600 5550
+Connection ~ 13450 5400
+Wire Wire Line
+	13450 5400 13450 5550
+Connection ~ 1850 3650
+Wire Wire Line
+	1850 3650 1850 3900
+Wire Wire Line
+	1550 1050 1550 1500
+Text GLabel 1550 1050 2    50   Input ~ 0
+POWER-IN+
+Text GLabel 1150 1050 0    50   Input ~ 0
+POWER-IN-
+Connection ~ 1150 3550
+Wire Wire Line
+	1150 3550 1150 2950
+Wire Wire Line
+	1150 1050 1150 1500
 $EndSCHEMATC

Commit message: second version, in progress
Parts:
- removed SW1, SW2, SW3, SW4, SW5, SW6, SW7: SW_DIP_x01, Button_Switch_THT:SW_DIP_SPSTx01_Slide_9.78x4.72mm_W7.62mm_P2.54mm, symbol Switch:SW_DIP_x01
- removed U11: LDH-45B-1050, OpenCelluloid:MeanWell-LDH-45B-1050, symbol ariadne:LDH-45B-1050
- removed U12, U15: Bridgelux-Vero-18, ariadne:Vero-18, symbol ariadne:Bridgelux-Vero-18
- removed U13, U6: Bridgelux-Vero-29, ariadne:Vero-29, symbol ariadne:Bridgelux-Vero-29
- removed U17: POTENTIOMETER, OpenCelluloid:PDB12-H4301-Potentiometer, symbol OpenSourceCelluloid:POTENTIOMETER
- removed U19, U23, U27: Heatsink-HP20S-CALBL-001, ariadne:Heatsink-HP20S-CALBL-001, symbol ariadne:Heatsink-HP20S-CALBL-001
- removed U2: Connector-LED-NILS, Connector_JST:JST_PH_B2B-PH-K_1x02_P2.00mm_Vertical, symbol ariadne:Connector-LED
- removed U22: Heatsink-NX301117, ariadne:Heatsink-NX301117, symbol ariadne:Heatsink-NX301117
- removed U28: Nils-Booster, Connector_JST:JST_PH_B4B-PH-K_1x04_P2.00mm_Vertical, symbol ariadne:Nils-Booster
- removed U7: OKI-78SR-5v, Converter_DCDC:Converter_DCDC_muRata_OKI-78SR_Vertical, symbol ariadne:OKI-78SR-5v
- removed U8, U9: Connector-LED, Connector_JST:JST_PH_B2B-PH-K_1x02_P2.00mm_Vertical, symbol ariadne:Connector-LED
- added C1: CP1_Small, Capacitor_THT:CP_Radial_D5.0mm_P2.00mm, symbol Device:CP1_Small
- added Murata-Ceramic-Capacitor-50v1-22uF1, Murata-Ceramic-Capacitor-50v1-22uF2, Murata-Ceramic-Capacitor-50v1-22uF3, Murata-Ceramic-Capacitor-50v1-22uF4, Murata-Ceramic-Capacitor-50v1-22uF5, Murata-Ceramic-Capacitor-50v1-22uF6: C, Capacitor_THT:C_Disc_D3.0mm_W1.6mm_P2.50mm, symbol Device:C
- added Q2: MMBT3904, Package_TO_SOT_SMD:SOT-23, symbol Transistor_BJT:MMBT3904
- added R12, R7, R8, R9: R, Resistor_THT:R_Axial_DIN0204_L3.6mm_D1.6mm_P7.62mm_Horizontal, symbol Device:R
- added U11: Noctua-NF-A4x10-Fan-mech, ariadne:Noctua-NF-A4x10, symbol ariadne:Noctua-NF-A4x10-Fan-mech
- added U13: Bridgelux-Vero-29-mech, ariadne:Vero-29-mech, symbol ariadne:Bridgelux-Vero-29-mech
- added U15: Bridgelux-Vero-18-mech, ariadne:Vero-18-mech, symbol ariadne:Bridgelux-Vero-18-mech
- added U18, U20: Meanwell-LDD-1200LW-connector, Connector_Molex:Molex_Micro-Fit_3.0_43650-0300_1x03_P3.00mm_Horizontal, symbol ariadne:Meanwell-LDD-1200LW-connector
- added U2: LDH-45B-1050-connector-slave, Connector_Molex:Molex_Micro-Fit_3.0_43650-0500_1x05_P3.00mm_Horizontal, symbol ariadne:LDH-45B-1050-connector
- added U23, U4: Connector-LED, Connector_JST:JST_PH_B2B-PH-K_1x02_P2.00mm_Vertical, symbol ariadne:Connector-LED
- added U3: LDH-45B-1050-connector-master, Connector_Molex:Molex_Micro-Fit_3.0_43650-0500_1x05_P3.00mm_Horizontal, symbol ariadne:LDH-45B-1050-connector
- added U5: OKI-78SR-12v, Converter_DCDC:Converter_DCDC_muRata_OKI-78SR_Vertical, symbol upuaut-rescue:OKI-78SR-12v-OpenSourceCelluloid
- added U6: OKI-78SR-5v, Converter_DCDC:Converter_DCDC_muRata_OKI-78SR_Vertical, symbol upuaut-rescue:OKI-78SR-5v-OpenSourceCelluloid
- added U8: LDH-45B-1050-mech, OpenCelluloid:MeanWell-LDH-45B-1050, symbol ariadne:LDH-45B-1050-mech
- R6: value 33k -> R
- U14: renamed from U18; footprint ariadne:Noctua-NF-A4x10 -> Connector_Molex:Molex_Micro-Fit_3.0_43650-0400_1x04_P3.00mm_Horizontal
- renumbered D2 to D1, D1 to D2, R7 to R10, R8 to R11, R9 to R13, R10 to R14, SW8 to SW1, SW9 to SW2, U3 to U10, U16 to U12, U5 to U16, U20 to U17, U21 to U19, U24 to U21, U25 to U22, U14 to U24, U26 to U25, U10 to U7, U4 to U9
Connections:
- net labels added: +24V, FAN-TACH, VIN+Master, VIN-Master
- net labels removed: POTI-45-B
- wire segments 170 -> 202
- no-connect marks 0 -> 1
Other:
- note added: "12V voltage regulator\n"
- note added: "3.3V voltage regulator\n\n"
- note added: "5V voltage regulator\n\n"
- note added: "Correct polarity protection\n"
- moved on the sheet: D1, D2, D3, R1, R10, R11, R13, R14

Commit message: BOM made at carla's
Parts:
- Q1: symbol ariadne:IRF5305-Reverse-Polarity -> ariadne-rescue:IRF5305-Reverse-Polarity-ariadne
- SW1, SW2: symbol ariadne:GB215AP -> ariadne-rescue:GB215AP-ariadne
- U1: symbol ariadne:Connector-POWER -> ariadne-rescue:Connector-POWER-ariadne
- U10: symbol ariadne:OKI-78SR-3.3_1.5-W36-C -> ariadne-rescue:OKI-78SR-3.3_1.5-W36-C-ariadne
- U11: symbol ariadne:Noctua-NF-A4x10-Fan-mech -> ariadne-rescue:Noctua-NF-A4x10-Fan-mech-ariadne
- U12, U17, U19, U21, U22, U25: symbol ariadne:01x15_2.50mm_HEADER_PIN -> ariadne-rescue:01x15_2.50mm_HEADER_PIN-ariadne
- U13: symbol ariadne:Bridgelux-Vero-29-mech -> ariadne-rescue:Bridgelux-Vero-29-mech-ariadne
- U14: symbol ariadne:Noctua-NF-A4x10-Fan -> ariadne-rescue:Noctua-NF-A4x10-Fan-ariadne
- U15: symbol ariadne:Bridgelux-Vero-18-mech -> ariadne-rescue:Bridgelux-Vero-18-mech-ariadne
- U16: symbol ariadne:ESP32-WROOM-32D -> ariadne-rescue:ESP32-WROOM-32D-ariadne
- U18, U20: symbol ariadne:Meanwell-LDD-1200LW-connector -> ariadne-rescue:Meanwell-LDD-1200LW-connector-ariadne
- U2, U3: symbol ariadne:LDH-45B-1050-connector -> ariadne-rescue:LDH-45B-1050-connector-ariadne
- U23, U4: symbol ariadne:Connector-LED -> ariadne-rescue:Connector-LED-ariadne
- U24: symbol ariadne:Meanwell-LDD-1200LW -> ariadne-rescue:Meanwell-LDD-1200LW-ariadne
- U5: symbol upuaut-rescue:OKI-78SR-12v-OpenSourceCelluloid -> ariadne-rescue:OKI-78SR-12v-OpenSourceCelluloid-upuaut-rescue
- U6: symbol upuaut-rescue:OKI-78SR-5v-OpenSourceCelluloid -> ariadne-rescue:OKI-78SR-5v-OpenSourceCelluloid-upuaut-rescue
- U7: symbol OpenSourceCelluloid:Power-Button -> ariadne-rescue:Power-Button-OpenSourceCelluloid
- U8: symbol ariadne:LDH-45B-1050-mech -> ariadne-rescue:LDH-45B-1050-mech-ariadne
- U9: symbol ariadne:CT2084-ND-DIP-SWITCH -> ariadne-rescue:CT2084-ND-DIP-SWITCH-ariadne
Changed lines of the file:
@@
 $EndDescr
 $Comp
-L ariadne:ESP32-WROOM-32D U16
+L ariadne-rescue:ESP32-WROOM-32D-ariadne U16
 U 1 1 5F84DC5D
 P 9300 1650
@@
 $EndComp
 $Comp
-L ariadne:Connector-POWER U1
+L ariadne-rescue:Connector-POWER-ariadne U1
 U 1 1 5F84F534
 P 1600 1600
@@
 $EndComp
 $Comp
-L ariadne:OKI-78SR-3.3_1.5-W36-C U10
+L ariadne-rescue:OKI-78SR-3.3_1.5-W36-C-ariadne U10
 U 1 1 5F84FE44
 P 5950 3900
@@
 $EndComp
 $Comp
-L ariadne:CT2084-ND-DIP-SWITCH U9
+L ariadne-rescue:CT2084-ND-DIP-SWITCH-ariadne U9
 U 1 1 5F850BB4
 P 5100 2050
@@
 $EndComp
 $Comp
-L ariadne:IRF5305-Reverse-Polarity Q1
+L ariadne-rescue:IRF5305-Reverse-Polarity-ariadne Q1
 U 1 1 5F853A6F
 P 2000 2900
@@
 $EndComp
 $Comp
-L ariadne:Meanwell-LDD-1200LW U24
+L ariadne-rescue:Meanwell-LDD-1200LW-ariadne U24
 U 1 1 5F86EF8E
 P 14350 4450
@@
 $EndComp
 $Comp
-L OpenSourceCelluloid:Power-Button U7
+L ariadne-rescue:Power-Button-OpenSourceCelluloid U7
 U 1 1 5F8ACF92
 P 2600 2200
@@
 $EndComp
 $Comp
-L ariadne:01x15_2.50mm_HEADER_PIN U12
+L ariadne-rescue:01x15_2.50mm_HEADER_PIN-ariadne U12
 U 1 1 5FA45304
 P 7650 1700
@@
 	8050 2350 8700 2350
 $Comp
-L ariadne:01x15_2.50mm_HEADER_PIN U17
+L ariadne-rescue:01x15_2.50mm_HEADER_PIN-ariadne U17
 U 1 1 5FA655F3
 P 11000 1700
@@
 	10900 2350 9900 2350
 $Comp
-L ariadne:01x15_2.50mm_HEADER_PIN U25
+L ariadne-rescue:01x15_2.50mm_HEADER_PIN-ariadne U25
 U 1 1 5FA8CCC2
 P 14600 7600
@@
 $EndComp
 $Comp
-L ariadne:01x15_2.50mm_HEADER_PIN U22
+L ariadne-rescue:01x15_2.50mm_HEADER_PIN-ariadne U22
 U 1 1 5FA8FF77
 P 13800 7600
@@
 $EndComp
 $Comp
-L ariadne:01x15_2.50mm_HEADER_PIN U21
+L ariadne-rescue:01x15_2.50mm_HEADER_PIN-ariadne U21
 U 1 1 5FA90DF1
 P 13000 7600
@@
 $EndComp
 $Comp
-L ariadne:01x15_2.50mm_HEADER_PIN U19
+L ariadne-rescue:01x15_2.50mm_HEADER_PIN-ariadne U19
 U 1 1 5FA915BA
 P 12150 7600
@@
 	14500 8150 14500 8250
 $Comp
-L ariadne:GB215AP SW1
+L ariadne-rescue:GB215AP-ariadne SW1
 U 1 1 5FAFA5B7
 P 10350 3550
@@
 	10600 4350 10950 4350
 $Comp
-L ariadne:GB215AP SW2
+L ariadne-rescue:GB215AP-ariadne SW2
 U 1 1 5FAFCC2F
 P 10350 4350
@@
 	9700 4350 10100 4350
 $Comp
-L ariadne:Noctua-NF-A4x10-Fan U14
+L ariadne-rescue:Noctua-NF-A4x10-Fan-ariadne U14
 U 1 1 5FB1994A
 P 8550 8450
@@
 $EndComp
 $Comp
-L upuaut-rescue:OKI-78SR-12v-OpenSourceCelluloid U5
+L ariadne-rescue:OKI-78SR-12v-OpenSourceCelluloid-upuaut-rescue U5
 U 1 1 5FB2E5DB
 P 2550 5100
@@
 $EndComp
 $Comp
-L upuaut-rescue:OKI-78SR-5v-OpenSourceCelluloid U6
+L ariadne-rescue:OKI-78SR-5v-OpenSourceCelluloid-upuaut-rescue U6
 U 1 1 5FB2E640
 P 2550 7000
@@
 NoConn ~ 2000 8700
 $Comp
-L ariadne:Connector-LED U4
+L ariadne-rescue:Connector-LED-ariadne U4
 U 1 1 5FBCC453
 P 2400 9650
@@
 	1800 8800 2000 8800
 $Comp
-L ariadne:LDH-45B-1050-connector U3
+L ariadne-rescue:LDH-45B-1050-connector-ariadne U3
 U 1 1 5FE3450C
 P 2200 8500
@@
 $EndComp
 $Comp
-L ariadne:LDH-45B-1050-connector U2
+L ariadne-rescue:LDH-45B-1050-connector-ariadne U2
 U 1 1 5FE434F1
 P 1900 10350
@@
 	1800 8900 2000 8900
 $Comp
-L ariadne:LDH-45B-1050-mech U8
+L ariadne-rescue:LDH-45B-1050-mech-ariadne U8
 U 1 1 5FE9BF38
 P 3000 10350
@@
 	2100 10850 2800 10850
 $Comp
-L ariadne:Meanwell-LDD-1200LW-connector U20
+L ariadne-rescue:Meanwell-LDD-1200LW-connector-ariadne U20
 U 1 1 5FF5322C
 P 12650 2700
@@
 $EndComp
 $Comp
-L ariadne:Meanwell-LDD-1200LW-connector U18
+L ariadne-rescue:Meanwell-LDD-1200LW-connector-ariadne U18
 U 1 1 5FF53985
 P 12050 4450
@@
 	12050 4750 14350 4750
 $Comp
-L ariadne:Connector-LED U23
+L ariadne-rescue:Connector-LED-ariadne U23
 U 1 1 5FFD7104
 P 13850 5400
@@
 	11200 2750 8800 2750
 $Comp
-L ariadne:Bridgelux-Vero-29-mech U13
+L ariadne-rescue:Bridgelux-Vero-29-mech-ariadne U13
 U 1 1 6011398A
 P 8000 10200
@@
 $EndComp
 $Comp
-L ariadne:Bridgelux-Vero-18-mech U15
+L ariadne-rescue:Bridgelux-Vero-18-mech-ariadne U15
 U 1 1 60114956
 P 9050 10200
@@
 $EndComp
 $Comp
-L ariadne:Noctua-NF-A4x10-Fan-mech U11
+L ariadne-rescue:Noctua-NF-A4x10-Fan-mech-ariadne U11
 U 1 1 60137C73
 P 6450 10250

Commit message: second version ready for layout
Parts:
- removed U1: Connector-POWER, OpenCelluloid:WAGO_PCB_Klemme_2Pol, symbol ariadne-rescue:Connector-POWER-ariadne
- removed U7: Power-Button, OpenCelluloid:WAGO_PCB_Klemme_3Pol, symbol ariadne-rescue:Power-Button-OpenSourceCelluloid
- added U1: POWER_CONNECTOR-DCJ250-20-B-K1-A, ariadne:POWER_JACK_DCJ250-20-B-K1-A, symbol ariadne:POWER_CONNECTOR-DCJ250-20-B-K1-A
- added U26: SWITCH_ROCKER-300DP3J1BLKM6QE, ariadne:SWITCH_ROCKER-300DP3J1BLKM6QE, symbol ariadne:SWITCH_ROCKER-300DP3J1BLKM6QE
- added U27, U7: LDH-65B-connector-master, Connector_Molex:Molex_Micro-Fit_3.0_43650-0400_1x04_P3.00mm_Horizontal, symbol ariadne:LDH-65B-connector
- added U28: Connector-LED, Connector_JST:JST_PH_B2B-PH-K_1x02_P2.00mm_Vertical, symbol ariadne-rescue:Connector-LED-ariadne
- added U29: LDH-65B-mech, ariadne:MeanWell-LDH-65, symbol ariadne:LDH-65B-mech
- Q1: footprint ariadne:IRF5305 -> Package_TO_SOT_THT:TO-220-3_Horizontal_TabDown
- Q2: footprint Package_TO_SOT_SMD:SOT-23 -> Package_TO_SOT_THT:TO-92
- U8: footprint OpenCelluloid:MeanWell-LDH-45B-1050 -> ariadne:MeanWell-LDH-45B-1050-ariadne
Connections:
- net labels added: 65B_OUT+, 65B_OUT-, BOARD_GND, LDH-65B-DIM
- wire segments 202 -> 200
- no-connect marks 1 -> 3
Changed lines of the file:
@@
 EELAYER 30 0
 EELAYER END
-$Descr A3 16535 11693
+$Descr A2 23386 16535
 encoding utf-8
 Sheet 1 1
@@
 $EndComp
 $Comp
-L ariadne-rescue:Connector-POWER-ariadne U1
-U 1 1 5F84F534
-P 1600 1600
-F 0 "U1" V 1604 1538 50  0000 L CNN
-F 1 "Connector-POWER" V 1695 1538 50  0000 L CNN
-F 2 "OpenCelluloid:WAGO_PCB_Klemme_2Pol" H 1600 1600 50  0001 C CNN
-F 3 "" H 1600 1600 50  0001 C CNN
-	1    1600 1600
-	-1   0    0    1
-$EndComp
-$Comp
 L ariadne-rescue:OKI-78SR-3.3_1.5-W36-C-ariadne U10
 U 1 1 5F84FE44
@@
 F 0 "Q1" H 2155 2946 50  0000 L CNN
 F 1 "IRF5305-Reverse-Polarity" H 2155 2855 50  0000 L CNN
-F 2 "ariadne:IRF5305" H 2150 2825 50  0001 L CIN
+F 2 "Package_TO_SOT_THT:TO-220-3_Horizontal_TabDown" H 2150 2825 50  0001 L CIN
 F 3 "http://www.irf.com/product-info/datasheets/data/irf7606pbf.pdf" V 1950 2900 50  0001 L CNN
 	1    2000 2900
@@
 	0    1    1    0
 $EndComp
-$Comp
-L ariadne-rescue:Power-Button-OpenSourceCelluloid U7
-U 1 1 5F8ACF92
-P 2600 2200
-F 0 "U7" V 2646 2222 50  0000 R CNN
-F 1 "Power-Button" V 2555 2222 50  0000 R CNN
-F 2 "OpenCelluloid:WAGO_PCB_Klemme_3Pol" H 2600 2200 50  0001 C CNN
-F 3 "" H 2600 2200 50  0001 C CNN
-	1    2600 2200
-	0    -1   -1   0
-$EndComp
-Connection ~ 1750 1450
-Wire Wire Line
-	1750 2200 2050 2200
-Wire Wire Line
-	1750 1450 1750 2050
-Wire Wire Line
-	1750 2050 2050 2050
-Connection ~ 1750 2050
-Wire Wire Line
-	1750 2050 1750 2200
 Wire Wire Line
 	2050 2350 2050 2700
@@
 Wire Wire Line
 	1350 3850 1350 3500
-Connection ~ 1350 1450
 $Comp
 L Device:D_Schottky D1
@@
 Wire Wire Line
 	1400 2900 1350 2900
-Connection ~ 1350 2900
-Wire Wire Line
-	1350 2900 1350 1450
 Text GLabel 3800 10850 2    50   Input ~ 0
 45B_OUT-
@@
 Text GLabel 8700 1550 0    50   Input ~ 0
 LDD_1200-DIM
-Text GLabel 2000 8600 0    50   Input ~ 0
-LDH_45B-DIM
 Text GLabel 8700 1450 0    50   Input ~ 0
 LDH_45B-DIM
@@
 Wire Wire Line
 	2050 3600 2050 3850
-Wire Wire Line
-	1750 1000 1750 1450
-Text GLabel 1750 1000 2    50   Input ~ 0
+Text GLabel 1650 1500 3    50   Input ~ 0
 POWER-IN+
-Text GLabel 1350 1000 0    50   Input ~ 0
+Text GLabel 1450 1500 3    50   Input ~ 0
 POWER-IN-
 Connection ~ 1350 3500
 Wire Wire Line
 	1350 3500 1350 2900
-Wire Wire Line
-	1350 1000 1350 1450
 $Comp
 L power:+24V #PWR06
@@
 Wire Notes Line
 	3400 750  550  750
-NoConn ~ 2000 8700
 $Comp
 L ariadne-rescue:Connector-LED-ariadne U4
@@
 F 0 "Q2" V 8835 6350 50  0000 C CNN
 F 1 "MMBT3904" V 8926 6350 50  0000 C CNN
-F 2 "Package_TO_SOT_SMD:SOT-23" H 8800 6275 50  0001 L CIN
+F 2 "Package_TO_SOT_THT:TO-92" H 8800 6275 50  0001 L CIN
 F 3 "https://www.fairchildsemi.com/datasheets/2N/2N3904.pdf" H 8600 6350 50  0001 L CNN
 	1    8600 6350
@@
 Wire Wire Line
 	9400 7350 10100 7350
-Wire Wire Line
-	1800 8900 1800 8800
-Wire Wire Line
-	1550 9000 2000 9000
-Wire Wire Line
-	1800 8800 2000 8800
 $Comp
 L ariadne-rescue:LDH-45B-1050-connector-ariadne U3
@@
 	-1   0    0    -1
 $EndComp
-Wire Wire Line
-	1800 8900 2000 8900
 $Comp
 L ariadne-rescue:LDH-45B-1050-mech-ariadne U8
@@
 F 0 "U8" H 3300 10515 50  0000 C CNN
 F 1 "LDH-45B-1050-mech" H 3300 10424 50  0000 C CNN
-F 2 "OpenCelluloid:MeanWell-LDH-45B-1050" H 3000 10350 50  0001 C CNN
+F 2 "ariadne:MeanWell-LDH-45B-1050-ariadne" H 3000 10350 50  0001 C CNN
 F 3 "" H 3000 10350 50  0001 C CNN
 	1    3000 10350
@@
 Text GLabel 1350 3850 2    50   Input ~ 0
 VIN-Master
-Text GLabel 1800 8800 0    50   Input ~ 0
-VIN-Master
-Text GLabel 1550 9000 0    50   Input ~ 0
-VIN+Master
 Wire Wire Line
 	2100 10450 2800 10450
@@
 	1    0    0    -1
 $EndComp
+$Comp
+L ariadne:SWITCH_ROCKER-300DP3J1BLKM6QE U26
+U 1 1 5FAE568D
+P 2300 2250
+F 0 "U26" V 2765 2225 50  0000 C CNN
+F 1 "SWITCH_ROCKER-300DP3J1BLKM6QE" V 2674 2225 50  0000 C CNN
+F 2 "ariadne:SWITCH_ROCKER-300DP3J1BLKM6QE" H 2300 2250 50  0001 C CNN
+F 3 "" H 2300 2250 50  0001 C CNN
+	1    2300 2250
+	0    -1   -1   0
+$EndComp
+Wire Wire Line
+	1750 2150 2050 2150
+NoConn ~ 2600 2250
+$Comp
+L ariadne-rescue:Connector-LED-ariadne U28
+U 1 1 5FB1745A
+P 2300 13300
+F 0 "U28" H 2350 13465 50  0000 C CNN
+F 1 "Connector-LED" H 2350 13374 50  0000 C CNN
+F 2 "Connector_JST:JST_PH_B2B-PH-K_1x02_P2.00mm_Vertical" H 2350 13283 50  0000 C CNN
+F 3 "" H 2300 13300 50  0001 C CNN
+	1    2300 13300
+	1    0    0    -1
+$EndComp
+Text GLabel 2100 12350 0    50   Input ~ 0
+VIN-Master
+Text GLabel 2100 12250 0    50   Input ~ 0
+VIN+Master
+Wire Notes Line
+	4550 14800 4550 11650
+Wire Notes Line
+	4550 11650 700  11650
+Wire Notes Line
+	700  11650 700  14800
+Wire Notes Line
+	700  14800 4550 14800
+$Comp
+L ariadne:LDH-65B-connector U27
+U 1 1 5FB30EF1
+P 2300 12150
+F 0 "U27" H 3028 11946 50  0000 L CNN
+F 1 "LDH-65B-connector-master" H 3028 11855 50  0000 L CNN
+F 2 "Connector_Molex:Molex_Micro-Fit_3.0_43650-0400_1x04_P3.00mm_Horizontal" H 2300 12150 50  0001 C CNN
+F 3 "" H 2300 12150 50  0001 C CNN
+	1    2300 12150
+	1    0    0    -1
+$EndComp
+Text GLabel 9900 1550 2    50   Input ~ 0
+LDH-65B-DIM
+Text GLabel 2100 12550 0    50   Input ~ 0
+LDH-65B-DIM
+Text GLabel 9950 2250 2    50   Input ~ 0
+BOARD_GND
+Text GLabel 2100 12450 0    50   Input ~ 0
+BOARD_GND
+$Comp
+L ariadne:LDH-65B-connector U7
+U 1 1 5FB4E63C
+P 1950 13900
+F 0 "U7" H 2192 14065 50  0000 C CNN
+F 1 "LDH-65B-connector-master" H 2192 13974 50  0000 C CNN
+F 2 "Connector_Molex:Molex_Micro-Fit_3.0_43650-0400_1x04_P3.00mm_Horizontal" H 1950 13900 50  0001 C CNN
+F 3 "" H 1950 13900 50  0001 C CNN
+	1    1950 13900
+	-1   0    0    -1
+$EndComp
+$Comp
+L ariadne:LDH-65B-mech U29
+U 1 1 5FB6658C
+P 2800 13900
+F 0 "U29" H 3100 14065 50  0000 C CNN
+F 1 "LDH-65B-mech" H 3100 13974 50  0000 C CNN
+F 2 "ariadne:MeanWell-LDH-65" H 2800 13900 50  0001 C CNN
+F 3 "" H 2800 13900 50  0001 C CNN
+	1    2800 13900
+	1    0    0    -1
+$EndComp
+Text GLabel 3600 14200 2    50   Input ~ 0
+65B_OUT+
+Text GLabel 3600 14300 2    50   Input ~ 0
+65B_OUT-
+Wire Wire Line
+	2150 14000 2600 14000
+Wire Wire Line
+	2150 14100 2600 14100
+Wire Wire Line
+	2150 14200 2600 14200
+Wire Wire Line
+	2150 14300 2600 14300
+Text GLabel 2550 13450 2    50   Input ~ 0
+65B_OUT-
+Text GLabel 2150 13450 0    50   Input ~ 0
+65B_OUT+
+Wire Wire Line
+	1650 1500 1750 1500
+Wire Wire Line
+	1750 1500 1750 2150
+Wire Wire Line
+	1350 1500 1350 2900
+Connection ~ 1350 2900
+Wire Wire Line
+	1350 1500 1450 1500
+$Comp
+L ariadne:POWER_CONNECTOR-DCJ250-20-B-K1-A U1
+U 1 1 5FBF2303
+P 1550 1250
+F 0 "U1" H 1322 1204 50  0000 R CNN
+F 1 "POWER_CONNECTOR-DCJ250-20-B-K1-A" H 1322 1295 50  0000 R CNN
+F 2 "ariadne:POWER_JACK_DCJ250-20-B-K1-A" H 1550 1250 50  0001 C CNN
+F 3 "" H 1550 1250 50  0001 C CNN
+	1    1550 1250
+	-1   0    0    1
+$EndComp
+NoConn ~ 1550 1000
+NoConn ~ 2000 8900
+Text GLabel 2000 8800 0    50   Input ~ 0
+BOARD_GND
+Text GLabel 2000 8600 0    50   Input ~ 0
+VIN+Master
+Text GLabel 2000 8700 0    50   Input ~ 0
+VIN-Master
+Text GLabel 2000 9000 0    50   Input ~ 0
+LDH_45B-DIM
 $EndSCHEMATC
