File: ariadne.sch (KiCad schematic (older format))
At the start: 57 parts, among them Q1 IRF5305-Reverse-Polarity, Q2 MMBT3904, SW1 GB215AP, SW2 GB215AP, U1 POWER_CONNECTOR-DCJ250-20-B-K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, U10 OKI-78SR-3.3_1.5-W36-C, U11 Noctua-NF-A4x10-Fan-mech, U12 01x15_2.50mm_HEADER_PIN, U13 Bridgelux-Vero-29-mech, U14 Noctua-NF-A4x10-Fan, U15 Bridgelux-Vero-18-mech, U16 ESP32-WROOM-32D, U17 01x15_2.50mm_HEADER_PIN, U18 Meanwell-LDD-1200LW-connector, U19 01x15_2.50mm_HEADER_PIN, U2 LDH-45B-1050-connector-slave, U20 Meanwell-LDD-1200LW-connector, U21 01x15_2.50mm_HEADER_PIN, U22 01x15_2.50mm_HEADER_PIN, U23 Connector-LED, U24 Meanwell-LDD-1200LW, U25 01x15_2.50mm_HEADER_PIN, U26 SWITCH_ROCKER-300DP3J1BLKM6QE, U27 LDH-65B-connector-master, U28 Connector-LED, U29 LDH-65B-mech, U3 LDH-45B-1050-connector-master, U4 Connector-LED, U5 OKI-78SR-12v, U6 OKI-78SR-5v, U7 LDH-65B-connector-master, U8 LDH-45B-1050-mech, U9 CT2084-ND-DIP-SWITCH

Commit message: Second version ordered
Parts:
- removed U19, U21, U22, U25: 01x15_2.50mm_HEADER_PIN, Connector_PinHeader_2.54mm:PinHeader_1x15_P2.54mm_Vertical, symbol ariadne-rescue:01x15_2.50mm_HEADER_PIN-ariadne
- added J1, J2, J3, J4: Conn_01x05_Male, Connector_PinHeader_2.54mm:PinHeader_1x05_P2.54mm_Vertical, symbol Connector:Conn_01x05_Male
- added U19: Noctua-NF-A4x10-Fan-mech-ariadne, ariadne:Noctua-NF-A4x10-mech, symbol ariadne-rescue:Noctua-NF-A4x10-Fan-mech-ariadne
- D1: value D_Schottky -> D_Zener
- U11: footprint ariadne:Noctua-NF-A4x10 -> ariadne:Noctua-NF-A4x10-mech
- U14: footprint Connector_Molex:Molex_Micro-Fit_3.0_43650-0400_1x04_P3.00mm_Horizontal -> Connector_PinHeader_2.54mm:PinHeader_1x04_P2.54mm_Vertical
Connections:
- wire segments 200 -> 159
Other:
- moved on the sheet: U11

Commit message: Ready for third version
Parts:
- U1: symbol ariadne:POWER_CONNECTOR-DCJ250-20-B-K1-A -> ariadne-rescue:POWER_CONNECTOR-DCJ250-20-B-K1-A-ariadne
- U26: symbol ariadne:SWITCH_ROCKER-300DP3J1BLKM6QE -> ariadne-rescue:SWITCH_ROCKER-300DP3J1BLKM6QE-ariadne
- U27, U7: symbol ariadne:LDH-65B-connector -> ariadne-rescue:LDH-65B-connector-ariadne
- U29: symbol ariadne:LDH-65B-mech -> ariadne-rescue:LDH-65B-mech-ariadne
Changed lines of the file:
@@
 $EndComp
 $Comp
-L ariadne:SWITCH_ROCKER-300DP3J1BLKM6QE U26
+L ariadne-rescue:SWITCH_ROCKER-300DP3J1BLKM6QE-ariadne U26
 U 1 1 5FAE568D
 P 2300 2250
@@
 	700  14800 4550 14800
 $Comp
-L ariadne:LDH-65B-connector U27
+L ariadne-rescue:LDH-65B-connector-ariadne U27
 U 1 1 5FB30EF1
 P 2300 12150
@@
 BOARD_GND
 $Comp
-L ariadne:LDH-65B-connector U7
+L ariadne-rescue:LDH-65B-connector-ariadne U7
 U 1 1 5FB4E63C
 P 1950 13900
@@
 $EndComp
 $Comp
-L ariadne:LDH-65B-mech U29
+L ariadne-rescue:LDH-65B-mech-ariadne U29
 U 1 1 5FB6658C
 P 2800 13900
@@
 	1350 1500 1450 1500
 $Comp
-L ariadne:POWER_CONNECTOR-DCJ250-20-B-K1-A U1
+L ariadne-rescue:POWER_CONNECTOR-DCJ250-20-B-K1-A-ariadne U1
 U 1 1 5FBF2303
 P 1550 1250

Commit message: Before carla leaves for HK
Parts:
- U24: symbol ariadne-rescue:Meanwell-LDD-1200LW-ariadne -> ariadne-rescue:Meanwell-LDD-1200LW-ariadne-ariadne-rescue
Connections:
- net LDD_1200_OUT+: now also U24.5 (VOUT+); no longer U24.13 (VOUT+)
- net LDD_1200_OUT-: now also U24.4 (VOUT-); no longer U24.12 (VOUT-)
- net at U24.2 (VIN-): now also U18.2 (VIN-)
- net at U18.1 (VIN+): now also U24.1 (VIN+); no longer U24.24 (VIN+)
- net at U18.3 (DIM): now also U24.3 (DIM)
Changed lines of the file:
@@
 $EndComp
 $Comp
-L ariadne-rescue:Meanwell-LDD-1200LW-ariadne U24
+L ariadne-rescue:Meanwell-LDD-1200LW-ariadne-ariadne-rescue U24
 U 1 1 5F86EF8E
 P 14350 4450
