File: _autosave-ariadne-v3.kicad_pcb (KiCad board)
At the start: 2 copper layers, 245 x 244.9 mm, 92 parts, among them J1 Conn_01x05_Male, J2 Conn_01x05_Male, J3 Conn_01x05_Male, J4 Conn_01x05_Male, J5 Conn_01x05_Male, Q1 IRF5305-Reverse-Polarity, U10 OKI-78SR-12v, U11 OKI-78SR-5v, U12 Meanwell-LDD-1200LW-connector, U14 Meanwell-LDD-1200LW-connector, U16 Connector-LED, U17 Connector-LED, U18 Meanwell-LDD-1200LW, U19 Meanwell-LDD-1200LW, U2 Meanwell-LDD-1200LW-connector, U20 Meanwell-LDD-1200LW-connector, U21 Meanwell-LDD-1200LW-connector, U22 Meanwell-LDD-1200LW-connector, U23 Meanwell-LDD-1200LW-connector, U24 ESP32-WROOM-32D, U25 Connector-LED, U26 Connector-LED, U27 Meanwell-LDD-1200LW, U28 Meanwell-LDD-1200LW, U29 Bridgelux-Vero-18-mech-v3-ari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, U3 POWER_CONNECTOR-DCJ250-20-B-K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, U31 Bridgelux-Vero-18-mech-v3-ari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, U32 Bridgelux-Vero-18-mech-v3-ari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, U33 Noctua-NF-A4x10-Simple-Fan-ar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, U34 Noctua-NF-A4x10-Simple-Fan-ar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, U35 Bridgelux-Vero-18-mech-v3-ari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, U36 Bridgelux-Vero-18-mech-v3-ari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, U37 heatsink, U38 heatsink, U39 heatsink, U40 heatsink, U41 heatsink, U42 heatsink, U43 Noctua-NF-A6x25Fan-mech-ariad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, U44 Noctua-NF-A6x25Fan-mech-ariad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, U5 Meanwell-LDD-1200LW-connector, U6 Connector-LED, U7 Connector-LED, U8 Meanwell-LDD-1200LW, U9 Meanwell-LDD-1200LW

Commit message: third version ready for production
Parts:
- added U1: Noctua-NF-A4x10-Simple-Fan-ariadne, Connector_JST:JST_XH_B2B-XH-AM_1x02_P2.50mm_Vertical, F.Cu at (67.8, 183.4)
- added U13: 12v-Connector, Connector_JST:JST_XH_B2B-XH-AM_1x02_P2.50mm_Vertical, F.Cu at (14.8, 67.7)
- added U15: 12v-Connector, Connector_JST:JST_XH_B2B-XH-AM_1x02_P2.50mm_Vertical, F.Cu at (64.3, 67.0)
- added U30: Bridgelux-Vero-18-mech-v3-ariadne, ariadne:Vero-18-mech, F.Cu at (-137.5, 16.2)
- added U4: Noctua-NF-A4x10-Simple-Fan-ariadne, Connector_JST:JST_XH_B2B-XH-AM_1x02_P2.50mm_Vertical, F.Cu at (67.8, 163.2)
- added U43: Noctua-NF-A4x10-Simple-Fan-ariadne, Connector_JST:JST_XH_B2B-XH-AM_1x02_P2.50mm_Vertical, F.Cu at (67.8, 144.4)
- added U44: Noctua-NF-A4x10-Simple-Fan-ariadne, Connector_JST:JST_XH_B2B-XH-AM_1x02_P2.50mm_Vertical, F.Cu at (16.0, 146.7)
- added U45: 12v-Connector_copy, Connector_JST:JST_XH_B2B-XH-AM_1x02_P2.50mm_Vertical, F.Cu at (16.2, 185.7)
- added U46: 12v-Connector_copy, Connector_JST:JST_XH_B2B-XH-AM_1x02_P2.50mm_Vertical, F.Cu at (42.1, 191.0)
- added U47: 12v-Connector_copy, Connector_JST:JST_XH_B2B-XH-AM_1x02_P2.50mm_Vertical, B.Cu at (43.0, 127.7)
