File: ariadne-v3.sch (KiCad schematic (older format))
At the start: 52 parts, among them J1 Conn_01x05_Male, J2 Conn_01x05_Male, J3 Conn_01x05_Male, J4 Conn_01x05_Male, J5 Conn_01x05_Male, Q1 IRF5305-Reverse-Polarity, U10 OKI-78SR-12v, U11 OKI-78SR-5v, U12 Meanwell-LDD-1200LW-connector, U14 Meanwell-LDD-1200LW-connector, U16 Connector-LED, U17 Connector-LED, U18 Meanwell-LDD-1200LW, U19 Meanwell-LDD-1200LW, U2 Meanwell-LDD-1200LW-connector, U20 Meanwell-LDD-1200LW-connector, U21 Meanwell-LDD-1200LW-connector, U22 Meanwell-LDD-1200LW-connector, U23 Meanwell-LDD-1200LW-connector, U24 ESP32-WROOM-32D, U25 Connector-LED, U26 Connector-LED, U27 Meanwell-LDD-1200LW, U28 Meanwell-LDD-1200LW, U29 Bridgelux-Vero-18-mech-v3-ari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, U3 POWER_CONNECTOR-DCJ250-20-B-K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, U30 Bridgelux-Vero-18-mech-v3-ari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, U31 Bridgelux-Vero-18-mech-v3-ari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, U32 Bridgelux-Vero-18-mech-v3-ari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, U33 Noctua-NF-A4x10-Simple-Fan-ar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, U34 Noctua-NF-A4x10-Simple-Fan-ar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, U35 Bridgelux-Vero-18-mech-v3-ari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, U36 Bridgelux-Vero-18-mech-v3-ari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, U37 heatsink, U38 heatsink, U39 heatsink, U40 heatsink, U41 heatsink, U42 heatsink, U43 Noctua-NF-A6x25Fan-mech-ariad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, U44 Noctua-NF-A6x25Fan-mech-ariad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, U5 Meanwell-LDD-1200LW-connector, U6 Connector-LED, U7 Connector-LED, U8 Meanwell-LDD-1200LW, U9 Meanwell-LDD-1200LW

Commit message: third version ready for production
Parts:
- removed U29, U30, U31, U32, U36: Bridgelux-Vero-18-mech-v3-ariadne, ariadne:Vero-18-mech, symbol ariadne-rescue:Bridgelux-Vero-18-mech-v3-ariadne
- removed U37, U38, U39, U40, U41, U42: heatsink, ariadne:Wakefield-heatsink, symbol ariadne-rescue:heatsink
- removed U43, U44: Noctua-NF-A6x25Fan-mech-ariadne, ariadne:Noctua-NF-A6x25-mech, symbol ariadne-rescue:Noctua-NF-A6x25Fan-mech-ariadne
- added U1, U4, U43, U44: Noctua-NF-A4x10-Simple-Fan-ariadne, Connector_JST:JST_XH_B2B-XH-AM_1x02_P2.50mm_Vertical, symbol ariadne-rescue:Noctua-NF-A4x10-Simple-Fan-ariadne
- added U13, U15: 12v-Connector, Connector_JST:JST_XH_B2B-XH-AM_1x02_P2.50mm_Vertical, symbol ariadne-rescue:12v-Connector
- added U29: Noctua-NF-A4x10-Fan-mech-ariadne, ariadne:Noctua-NF-A4x10, symbol ariadne-rescue:Noctua-NF-A4x10-Fan-mech-ariadne
- added U45, U47: 12v-Connector_copy, Connector_JST:JST_XH_B2B-XH-AM_1x02_P2.50mm_Vertical, symbol ariadne-rescue:12v-Connector_copy
- U12, U14, U2, U20, U21, U22, U23, U5: footprint Connector_Molex:Molex_Micro-Fit_3.0_43650-0300_1x03_P3.00mm_Horizontal -> Connector_Molex:Molex_Micro-Fit_3.0_43650-0315_1x03_P3.00mm_Vertical
- U18, U19, U27, U28, U8, U9: symbol ariadne-rescue:Meanwell-LDD-1200LW-ariadne -> ariadne-v3-rescue:Meanwell-LDD-1200LW-ariadne-ariadne-rescue
Connections:
- net labels added: FAN1+, FAN1-, FAN2+, FAN2-
- no-connect marks 7 -> 1
Other:
- moved on the sheet: U33, U34
